File: hardware/Araneae/Araneae.kicad_sch (KiCad schematic)
At the start: 0 parts

Commit message: Add CI workflow for PCB checks and artifact generation
- Created a GitHub Actions workflow (`ci.yml`) to automate hardware checks including ERC, DRC, and plot generation for KiCad projects.
- Added a new footprint for the SON50P200X200X80-9N component in `SON50P200X200X80-9N.kicad_mod`.
- Introduced a new symbol for the TPS22965DSGR component in `TPS22965DSGR.kicad_sym`.
- Added a configuration file `kibot.yaml` for generating fabrication files and other outputs.
Other:
- sheet CM4 ports: added TMP1_SCL, TMP1_SDA, TMP2_SCL, TMP2_SDA, WATCHDOG_WDI, {DIS}, {ETH_Boost}, {ETH}, {HDMI}, {SD}, {SSD}, {UPS}, {USB_HUB}; removed none
- sheet Display Conn ports: added {DIS}; removed none
- sheet Ethernet Boost ports: added {ETH_Boost}, {ETH}; removed none
- sheet HDMI ports: added {HDMI}; removed none
- sheet Micro SD ports: added {SD}; removed none
- sheet RJ-45 ports: added {ETH}; removed none
- sheet SSD PCle ports: added {SSD_Sec}, {SSD}; removed none
- sheet SSD Support and Security ports: added {SSD_Sec}; removed none
- sheet System Supervision ports: added TMP1_SCL, TMP1_SDA, TMP2_SCL, TMP2_SDA, WATCHDOG_WDI; removed none
- sheet UPS Subsystem ports: added {UPS}; removed none
- sheet USB Hub ports: added {USBA1_HUB}, {USBA2_HUB}, {USBA3_HUB}, {USBC_HUB}, {USB_HUB}; removed CM4_USB_D+, CM4_USB_D-, USBA1_D+, USBA1_D-, USBA1_FAULT_N, USBA1_PWR_EN, USBA2_D+, USBA2_D-, USBA2_FAULT_N, USBA2_PWR_EN, USBA3_D+, USBA3_D-, USBA3_FAULT_N, USBA3_PWR_EN, USBC_D+, USBC_D-, USBC_FAULT_N, USBC_PWR_EN, USB_HUB_RESET_N
- sheet USB-A ports: added {USBA1_HUB}, {USBA2_HUB}, {USBA3_HUB}; removed none
- sheet USB-C ports: added {USBC_HUB}; removed USBC_D+, USBC_D-, USBC_FAULT_N, USBC_PWR_EN
- note added: "Global Nets Only"
- company: (none) -> Matheus Henrique(Aka: TheusHen)
- title: (none) -> Araneae
