File: hardware/Araneae/cm4.kicad_sch (KiCad schematic)
At the start: 3 parts, among them X1 DF40HC_3.0_-100DS-0.4V_58, X2 DF40HC_3.0_-100DS-0.4V_58

Commit message: Add CI workflow for PCB checks and artifact generation
- Created a GitHub Actions workflow (`ci.yml`) to automate hardware checks including ERC, DRC, and plot generation for KiCad projects.
- Added a new footprint for the SON50P200X200X80-9N component in `SON50P200X200X80-9N.kicad_mod`.
- Introduced a new symbol for the TPS22965DSGR component in `TPS22965DSGR.kicad_sym`.
- Added a configuration file `kibot.yaml` for generating fabrication files and other outputs.
Parts:
- R25: footprint (none) -> Resistor_SMD:R_0805_2012Metric
- X1, X2: footprint DF40HC_3.0_-100DS-0.4V_58:HRS_DF40HC_3.0_-100DS-0.4V_58 -> OPL:HRS_DF40HC_3.0_-100DS-0.4V_58
Connections:
- net +1V8: now also X1.94, X1.96
- net CM4_USB_D+ renamed CM4_USB_D_P
- net CM4_USB_D- renamed CM4_USB_D_N
- net ETH1_MX1+ renamed ETH1_MX1_P
- net ETH1_MX1- renamed ETH1_MX1_N
- net ETH1_MX2+ renamed ETH1_MX2_P
- net ETH1_MX2- renamed ETH1_MX2_N
- net ETH1_MX3+ renamed ETH1_MX3_P
- net ETH1_MX3- renamed ETH1_MX3_N
- net ETH1_MX4+ renamed ETH1_MX4_P
- net ETH1_MX4- renamed ETH1_MX4_N
- no-connect marks 32 -> 52
Other:
- company: (none) -> Matheus Henrique(Aka: TheusHen)
- title: (none) -> Araneae
- moved on the sheet: R25
Changed lines of the file:
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@@
 	(generator_version "10.0")
 	(paper "A4")
+	(title_block
+		(title "Araneae")
+		(date "2026-05-02")
+		(rev "0.1")
+		(company "Matheus Henrique(Aka: TheusHen)")
+		(comment 1 "dev@theushen.works")
+		(comment 3 "z2mCL9YdujNw7uhfDBhsiKtEFSAYvfbvY")
+		(comment 4 "Donate(Monero): 8A8gezqQ4tuVAPWAYUKB7rB5NRLFWE3RsXWFQLKh3jVAceb9pG4VjA8ApUd8DM")
+	)
