File: hardware/Araneae/headers.kicad_sch (KiCad schematic)
At the start: 66 parts, among them J10 Conn_01x04, J11 Conn_01x04, J7 Conn_01x04, J8 Conn_01x04, J9 Conn_02x13_Top_Bottom

Commit message: Add CI workflow for PCB checks and artifact generation
- Created a GitHub Actions workflow (`ci.yml`) to automate hardware checks including ERC, DRC, and plot generation for KiCad projects.
- Added a new footprint for the SON50P200X200X80-9N component in `SON50P200X200X80-9N.kicad_mod`.
- Introduced a new symbol for the TPS22965DSGR component in `TPS22965DSGR.kicad_sym`.
- Added a configuration file `kibot.yaml` for generating fabrication files and other outputs.
Parts:
- D21: value D_TVS -> TVS_3V3; footprint (none) -> Diode_SMD:D_SOD-323
- D22: value D_TVS -> ESD_5V; footprint (none) -> Diode_SMD:D_SOD-323
- D23, D24, D26, D28, D29, D30, D32, D33: value D_TVS -> ESD_3V3; footprint (none) -> Diode_SMD:D_SOD-323
- D25, D27, D31: value D_TVS -> TVS_12V; footprint (none) -> Diode_SMD:D_SMF
- F3: value Polyfuse -> 500mA; footprint (none) -> Fuse:Fuse_1206_3216Metric
- F4: value Polyfuse -> TVS_5V; footprint (none) -> Fuse:Fuse_1206_3216Metric
- F5: value Polyfuse -> 1.5A; footprint (none) -> Fuse:Fuse_1812_4532Metric
- F6, F7: value Polyfuse -> 1A; footprint (none) -> Fuse:Fuse_1812_4532Metric
- J10: renamed from J9; footprint (none) -> Connector_IDC:IDC-Header_2x13_P2.54mm_Horizontal
- J11: renamed from J10; footprint (none) -> Connector_PinHeader_2.54mm:PinHeader_1x04_P2.54mm_Vertical
- J12: renamed from J11; footprint (none) -> Connector_PinHeader_2.54mm:PinHeader_1x04_P2.54mm_Vertical
- J8: renamed from J7; footprint (none) -> Connector_PinHeader_2.54mm:PinHeader_1x04_P2.54mm_Vertical
- J9: renamed from J8; footprint (none) -> Connector_PinHeader_2.54mm:PinHeader_1x04_P2.54mm_Vertical
- R52: renamed from R51; footprint (none) -> Resistor_SMD:R_0603_1608Metric
- R53: renamed from R52; footprint (none) -> Resistor_SMD:R_0603_1608Metric
- R54: renamed from R53; footprint (none) -> Resistor_SMD:R_0603_1608Metric
- R55: renamed from R54; footprint (none) -> Resistor_SMD:R_0603_1608Metric
- R56: renamed from R55; footprint (none) -> Resistor_SMD:R_0603_1608Metric
- R57: renamed from R56; footprint (none) -> Resistor_SMD:R_0603_1608Metric
- R58: renamed from R57; footprint (none) -> Resistor_SMD:R_0603_1608Metric
- R59: renamed from R58; footprint (none) -> Resistor_SMD:R_0603_1608Metric
- R60: renamed from R59; footprint (none) -> Resistor_SMD:R_0603_1608Metric
- R61: renamed from R60; footprint (none) -> Resistor_SMD:R_0603_1608Metric
- R62: renamed from R61; footprint (none) -> Resistor_SMD:R_0603_1608Metric
- R63: renamed from R62; footprint (none) -> Resistor_SMD:R_0603_1608Metric
- R64: renamed from R63; footprint (none) -> Resistor_SMD:R_0603_1608Metric
- R65: renamed from R64; footprint (none) -> Resistor_SMD:R_0603_1608Metric
- R66: renamed from R65; footprint (none) -> Resistor_SMD:R_0603_1608Metric
- R67: renamed from R66; footprint (none) -> Resistor_SMD:R_0603_1608Metric
- R68: renamed from R67; footprint (none) -> Resistor_SMD:R_0603_1608Metric
- R69: renamed from R68; footprint (none) -> Resistor_SMD:R_0603_1608Metric
- R70: renamed from R69; footprint (none) -> Resistor_SMD:R_0603_1608Metric
- R71: renamed from R70; footprint (none) -> Resistor_SMD:R_0603_1608Metric
- R72: renamed from R71; footprint (none) -> Resistor_SMD:R_0603_1608Metric
- R73: renamed from R72; footprint (none) -> Resistor_SMD:R_0603_1608Metric
- R74: renamed from R73; footprint (none) -> Resistor_SMD:R_0603_1608Metric
- R75: renamed from R74; footprint (none) -> Resistor_SMD:R_0603_1608Metric
- R76: renamed from R75; footprint (none) -> Resistor_SMD:R_0603_1608Metric
- R77: renamed from R76; footprint (none) -> Resistor_SMD:R_0603_1608Metric
- R78: renamed from R77; footprint (none) -> Resistor_SMD:R_0603_1608Metric
- R79: renamed from R78; footprint (none) -> Resistor_SMD:R_0603_1608Metric
- R80: renamed from R79; footprint (none) -> Resistor_SMD:R_0603_1608Metric
- R81: renamed from R80; footprint (none) -> Resistor_SMD:R_0603_1608Metric
- R82: renamed from R81; footprint (none) -> Resistor_SMD:R_0603_1608Metric
- R83: renamed from R82; footprint (none) -> Resistor_SMD:R_0603_1608Metric
- R84: renamed from R83; footprint (none) -> Resistor_SMD:R_0603_1608Metric
- R85: renamed from R84; footprint (none) -> Resistor_SMD:R_0603_1608Metric
- R86: renamed from R85; footprint (none) -> Resistor_SMD:R_0603_1608Metric
- R87: renamed from R86; footprint (none) -> Resistor_SMD:R_0603_1608Metric
- R88: renamed from R87; footprint (none) -> Resistor_SMD:R_0603_1608Metric
- R89: renamed from R88; footprint (none) -> Resistor_SMD:R_0603_1608Metric
- R90: renamed from R89; footprint (none) -> Resistor_SMD:R_0603_1608Metric
- TP1, TP2, TP3, TP4: footprint (none) -> TestPoint:TestPoint_Pad_D1.5mm
Connections:
- net +3V3: now also R58.2, R59.2
- net GND: no longer R58.2, R59.2
Other:
- note added: "2xDelta AFB1212SHE PWM 120x38mm"
- note removed: "2xDelta AUB0912VH"
- company: (none) -> Matheus Henrique(Aka: TheusHen)
- title: (none) -> Araneae
- moved on the sheet: D22, D29, D33
