File: hardware/Araneae/power.kicad_sch (KiCad schematic)
At the start: 42 parts, among them IC1 MP1584EN-LF-Z, IC2 MP1584EN-LF-Z, J6 Barrel_Jack, U12 TPS54331DG4

Commit message: Add CI workflow for PCB checks and artifact generation
- Created a GitHub Actions workflow (`ci.yml`) to automate hardware checks including ERC, DRC, and plot generation for KiCad projects.
- Added a new footprint for the SON50P200X200X80-9N component in `SON50P200X200X80-9N.kicad_mod`.
- Introduced a new symbol for the TPS22965DSGR component in `TPS22965DSGR.kicad_sym`.
- Added a configuration file `kibot.yaml` for generating fabrication files and other outputs.
Parts:
- C32: renamed from C33; footprint (none) -> Capacitor_SMD:C_0805_2012Metric
- C33: renamed from C34; footprint (none) -> Capacitor_SMD:C_0805_2012Metric
- C34: renamed from C35; footprint (none) -> Capacitor_SMD:C_0603_1608Metric
- C35: renamed from C36; footprint (none) -> Capacitor_SMD:C_0805_2012Metric
- C36: renamed from C37; footprint (none) -> Capacitor_SMD:C_0603_1608Metric
- C37: renamed from C38; footprint (none) -> Capacitor_SMD:C_0603_1608Metric
- C38: renamed from C39; footprint (none) -> Capacitor_SMD:C_0603_1608Metric
- C39: renamed from C40; footprint (none) -> Capacitor_SMD:C_0603_1608Metric
- C40: renamed from C41; footprint (none) -> Capacitor_SMD:C_0603_1608Metric
- C41: renamed from C42; footprint (none) -> Capacitor_SMD:C_1206_3216Metric
- C42: renamed from C43; footprint (none) -> Capacitor_SMD:C_1206_3216Metric
- C43: renamed from C44; footprint (none) -> Capacitor_SMD:C_0603_1608Metric
- C44: renamed from C45; footprint (none) -> Capacitor_SMD:C_0805_2012Metric
- C45: renamed from C46; footprint (none) -> Capacitor_SMD:C_0603_1608Metric
- C46: renamed from C47; footprint (none) -> Capacitor_SMD:C_0603_1608Metric
- C47: renamed from C48; footprint (none) -> Capacitor_SMD:C_0603_1608Metric
- C48: renamed from C49; footprint (none) -> Capacitor_SMD:C_0805_2012Metric
- C49: renamed from C50; footprint (none) -> Capacitor_SMD:C_0805_2012Metric
- D17, D18, D19: footprint (none) -> Diode_SMD:D_SMA
- D20: value D_Schottky -> SS34; footprint (none) -> Diode_SMD:D_SMA
- F2: value Polyfuse -> 3A; footprint (none) -> Fuse:Fuse_1812_4532Metric
- IC1, IC2: footprint MP1584EN-LF-Z:SOIC127P600X170-9N -> OPL:SOIC127P600X170-9N
- J7: renamed from J6; footprint (none) -> Connector_BarrelJack:BarrelJack_CUI_PJ-102AH_Horizontal
- L2, L3: footprint (none) -> Inductor_SMD:L_7.3x7.3_H4.5
- L4: footprint (none) -> Inductor_SMD:L_10.4x10.4_H4.8
- R41: renamed from R40; footprint (none) -> Resistor_SMD:R_0603_1608Metric
- R42: renamed from R41; footprint (none) -> Resistor_SMD:R_0603_1608Metric
- R43: renamed from R42; footprint (none) -> Resistor_SMD:R_0603_1608Metric
- R44: renamed from R43; footprint (none) -> Resistor_SMD:R_0603_1608Metric
- R45: renamed from R44; footprint (none) -> Resistor_SMD:R_0603_1608Metric
- R46: renamed from R45; footprint (none) -> Resistor_SMD:R_0603_1608Metric
- R47: renamed from R46; footprint (none) -> Resistor_SMD:R_0603_1608Metric
- R48: renamed from R47; footprint (none) -> Resistor_SMD:R_0603_1608Metric
- R49: renamed from R48; footprint (none) -> Resistor_SMD:R_0603_1608Metric
- R50: renamed from R49; footprint (none) -> Resistor_SMD:R_0603_1608Metric
- R51: renamed from R50; footprint (none) -> Resistor_SMD:R_0603_1608Metric
- U12: footprint TPS54331DG4:SOIC127P599X175-8N -> OPL:SOIC127P599X175-8N
Connections:
- net 19V: now also F2.1; no longer D16.1 (A1), D17.1 (K), F2.2, J7.1
- net GND: no longer F2.1
- new net: D16.1 (A1), D17.1 (K), F2.2, J7.1
Other:
- company: (none) -> Matheus Henrique(Aka: TheusHen)
- title: (none) -> Araneae
