File: hardware/Araneae/supervision.kicad_sch (KiCad schematic)
At the start: 17 parts, among them U16 TPS3430WDRCR, U17 TLV809I50DBZT, U18 TLV809K33DBZR, U19 TMP117AIDRVR, U20 TMP117AIDRVR

Commit message: Add CI workflow for PCB checks and artifact generation
- Created a GitHub Actions workflow (`ci.yml`) to automate hardware checks including ERC, DRC, and plot generation for KiCad projects.
- Added a new footprint for the SON50P200X200X80-9N component in `SON50P200X200X80-9N.kicad_mod`.
- Introduced a new symbol for the TPS22965DSGR component in `TPS22965DSGR.kicad_sym`.
- Added a configuration file `kibot.yaml` for generating fabrication files and other outputs.
Parts:
- C64: renamed from C65; footprint (none) -> Capacitor_SMD:C_0603_1608Metric
- C65: renamed from C66; footprint (none) -> Capacitor_SMD:C_0603_1608Metric
- C66: renamed from C67; footprint (none) -> Capacitor_SMD:C_0603_1608Metric
- C67: renamed from C68; footprint (none) -> Capacitor_SMD:C_0603_1608Metric
- R92: renamed from R91; footprint (none) -> Resistor_SMD:R_0603_1608Metric
- R93: renamed from R92; footprint (none) -> Resistor_SMD:R_0603_1608Metric
- R94: renamed from R93; footprint (none) -> Resistor_SMD:R_0603_1608Metric
- R95: renamed from R94; footprint (none) -> Resistor_SMD:R_0603_1608Metric
- R96: renamed from R95; footprint (none) -> Resistor_SMD:R_0603_1608Metric
- U16: footprint TPS3430WDRCR:VREG_V62_16624-01YE -> OPL:VREG_V62_16624-01YE
- U17: footprint TLV809I50DBZT:SOT95P280X145-3N -> OPL:SOT95P280X145-3N
- U18: footprint TLV809K33DBZR:SOT95P280X145-3N -> OPL:SOT95P280X145-3N
- U19, U20: footprint TMP117AIDRVR:SON65P200X200X80-7N -> OPL:SON65P200X200X80-7N
Connections:
- net +3V3: now also R93.1, R94.1, R95.2, R96.1, U20.4 (ADD0)
- net GND: no longer U20.4 (ADD0)
- net TMP1_SCL: now also R93.2, U19.1 (SCL); no longer R93.1
- net TMP1_SDA: now also R94.2, U19.6 (SDA); no longer R94.1
- net TMP2_SCL: now also U20.1 (SCL)
- net TMP2_SDA: now also R96.2, U20.6 (SDA); no longer R96.1
Other:
- company: (none) -> Matheus Henrique(Aka: TheusHen)
- title: (none) -> Araneae
- moved on the sheet: R93, R94, R95, R96
