File: hardware/Araneae/ups.kicad_sch (KiCad schematic)
At the start: 58 parts, among them Q1 PMOS, Q2 NMOS, Q3 PMOS, Q4 NMOS, U1 LTC4412xS6, U2 ISL94202IRTZ, U3 IRLR7843, U4 IRLR7843, U5 LTC4015EUHF

Commit message: Add CI workflow for PCB checks and artifact generation
- Created a GitHub Actions workflow (`ci.yml`) to automate hardware checks including ERC, DRC, and plot generation for KiCad projects.
- Added a new footprint for the SON50P200X200X80-9N component in `SON50P200X200X80-9N.kicad_mod`.
- Introduced a new symbol for the TPS22965DSGR component in `TPS22965DSGR.kicad_sym`.
- Added a configuration file `kibot.yaml` for generating fabrication files and other outputs.
Parts:
- removed R13: 10k, symbol Device:R
- removed R16: 5mΩ, symbol Device:R_Shunt
- removed R19: 301k, symbol Device:R
- removed R24: 15mΩ, symbol Device:R_Shunt
- added C85, C86, C87: 100nF, Capacitor_SMD:C_0603_1608Metric, symbol Device:C
- added R120, R121: 4.7k, Resistor_SMD:R_0603_1608Metric, symbol Device:R
- added R16: 10mΩ, Resistor_SMD:R_2512_6332Metric, symbol Device:R
- added R24: 30mΩ, Resistor_SMD:R_2512_6332Metric, symbol Device:R
- BT1, BT2: footprint 1048:BAT_1048 -> OPL:BAT_1048
- C1, C11, C12, C14, C15, C18, C2, C3, C7, C9: footprint (none) -> Capacitor_SMD:C_0603_1608Metric
- C10, C16, C17, C8: footprint (none) -> Capacitor_SMD:C_0805_2012Metric
- C13: value 1µF -> 2.2µF; footprint (none) -> Capacitor_SMD:C_0603_1608Metric
- C4: renamed from C5; footprint (none) -> Capacitor_SMD:C_0603_1608Metric
- C5: renamed from C6; footprint (none) -> Capacitor_SMD:C_0603_1608Metric
- C6: renamed from C4; footprint (none) -> Capacitor_SMD:C_0603_1608Metric
- D2: footprint (none) -> LED_SMD:LED_0805_2012Metric
- L1: footprint (none) -> Inductor_SMD:L_10.4x10.4_H4.8
- Q1, Q2, Q3, Q4: footprint (none) -> Package_TO_SOT_SMD:SOT-23
- R1: footprint (none) -> Resistor_SMD:R_2512_6332Metric
- R10, R12, R14, R17, R18, R2, R21, R22, R23, R3, R4, R5, R7, R8, R9, TH1, TH2: footprint (none) -> Resistor_SMD:R_0603_1608Metric
- R11: value 100k -> 10k; footprint (none) -> Resistor_SMD:R_0603_1608Metric
- R15: value 95.3k -> 10k; footprint (none) -> Resistor_SMD:R_0603_1608Metric
- R20: value 301k -> 124k; footprint (none) -> Resistor_SMD:R_0603_1608Metric
- R6: footprint (none) -> Resistor_SMD:R_0805_2012Metric
- U2: footprint ISL94202IRTZ:QFN40P600X600X80-49N -> OPL:QFN40P600X600X80-49N
- U3, U4: footprint IRLR7843:TO252 -> OPL:TO252
- U5: footprint LTC4015EUHF:QFN50P700X500X80-39N -> OPL:QFN50P700X500X80-39N
Connections:
- net CSN is gone; now on net BAT_P: U5.19 (CSN)
- net +12V: no longer U2.10 (CB4)
- net +12V_BAT: now also U2.10 (CB4)
- net +3V3: no longer R14.1
- net 12V_SYSTEM: now also C85.1
- net 19V: now also U5.32 (CLN), U5.33 (CLP), R16.1, R16.2
- net CCREFM: now also R18.1, U5.16 (CCREFM)
- net CCREFP: now also R18.2, U5.17 (CCREFP); no longer R18.1
- net CSP: now also L1.1, C86.2, R24.1; no longer U5.15 (CSPM5)
- net DVCC: no longer U5.1 (CELLS1), U5.38 (CELLS0)
- net GND: now also U5.1 (CELLS1), C87.2; no longer R10.1, R11.1, R12.1, U5.30 (SYSM5)
- net UPS1_N1: now also U2.14 (CB2)
- net UPS2_N2: no longer U2.14 (CB2)
- net UPS_SCL: now also R120.2
- net UPS_SDA: now also U2.26 (SDAI), R121.2
- net at U2.36 (RGO): now also R10.1, R11.1, R12.1, R14.1, C87.1, R120.1, R121.1
- net BAT+ renamed BAT_P
- net BAT_P: now also R24.2
- new net: C86.1, U5.15 (CSPM5)
- new net: C85.2, U5.30 (SYSM5)
- no-connect marks 5 -> 6
Other:
- note added: "1.2 × (124k + 10k) / 10k ≈ 16.1V"
- note added: "Official Quality Certified LFP 26650 3.2v 2500Mh Grade A_P LiFePO4 Battery Rechargeable Battery Golfcarts RV Deep Cycle Battery"
- note removed: "2.494 × (301k + 95.3k) / 95.3k ≈ 10.4V"
- note removed: "Official Quality Certified LFP 26650 3.2v 2500Mh Grade A+ LiFePO4 Battery Rechargeable Battery Golfcarts RV Deep Cycle Battery"
- company: (none) -> Matheus Henrique(Aka: TheusHen)
- title: (none) -> Araneae
- moved on the sheet: C6, Q2, Q4, R1, R14, R6
